File: CoinLogger.sch (EAGLE design)
At the start: 17 parts, among them IC1 TINY11S, U4 LIS331

Commit message: Board is now v1.1
Parts:
- removed JP1: USB_MICROB_PLUG, SparkFun:USB_MICROB_PLUG
- added X1: USB-MICROB, SparkFun:USB-MICROB
- renumbered BAT2 to BAT1
Connections:
- net GND: now also X1.GND; no longer JP1.GND
- net N$2: now also X1.D+; no longer JP1.D+
- net N$6: now also IC1.(AIN0)PB0, JP2.1; no longer IC1.(AIN1)PB1, JP2.2
- net N$7: now also IC1.(AIN1)PB1, JP2.2; no longer IC1.(AIN0)PB0, JP2.1
- net N$8: now also X1.D-; no longer JP1.D-
Other:
- note added: "PB0: MOSI"
- note added: "PB1: MISO"
- note added: "PB2: SCK"
- note added: "PB3: CS"
Changed lines of the file:
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@@
 <part name="GND7" library="supply1" deviceset="GND" device=""/>
 <part name="GND2" library="supply1" deviceset="GND" device=""/>
-<part name="BAT2" library="SparkFun" deviceset="BATTERY" device="20SMD"/>
 <part name="JP2" library="SparkFun" deviceset="M06" device="1X06-SMD_EDGE_FEMALE"/>
 <part name="U4" library="SparkFun" deviceset="LIS331" device=""/>
 <part name="GND3" library="supply1" deviceset="GND" device=""/>
-<part name="JP1" library="SparkFun" deviceset="USB_MICROB_PLUG" device=""/>
 <part name="R1" library="SparkFun" deviceset="RESISTOR" device="0402-RES" value="68"/>
 <part name="R2" library="SparkFun" deviceset="RESISTOR" device="0402-RES" value="68"/>
@@
 <part name="LED1" library="SparkFun" deviceset="LED" device="0603"/>
 <part name="GND9" library="supply1" deviceset="GND" device=""/>
+<part name="X1" library="SparkFun" deviceset="USB" device="-MICROB"/>
+<part name="BAT1" library="SparkFun" deviceset="BATTERY" device="20SMD"/>
 </parts>
 <sheets>
@@
 <text x="83.82" y="-22.86" size="1.778" layer="97">Might also make a version with uSD card, but they're so power hungry...</text>
 <text x="83.82" y="-25.4" size="1.778" layer="97">Uses CR2032 coin cell</text>
+<text x="33.02" y="78.74" size="1.778" layer="97">PB0: MOSI</text>
+<text x="33.02" y="76.2" size="1.778" layer="97">PB1: MISO</text>
+<text x="33.02" y="73.66" size="1.778" layer="97">PB2: SCK</text>
+<text x="33.02" y="71.12" size="1.778" layer="97">PB3: CS</text>
 </plain>
 <instances>
@@
 <instance part="GND7" gate="1" x="22.86" y="7.62"/>
 <instance part="GND2" gate="1" x="15.24" y="68.58"/>
-<instance part="BAT2" gate="G$1" x="10.16" y="76.2"/>
 <instance part="JP2" gate="G$1" x="83.82" y="53.34" rot="MR0"/>
 <instance part="U4" gate="G$1" x="-2.54" y="-12.7"/>
 <instance part="GND3" gate="1" x="-27.94" y="-30.48"/>
-<instance part="JP1" gate="G$1" x="81.28" y="73.66" smashed="yes">
-<attribute name="NAME" x="76.454" y="81.788" size="1.778" layer="95"/>
-<attribute name="VALUE" x="88.9" y="73.914" size="1.778" layer="96"/>
-</instance>
 <instance part="R1" gate="G$1" x="60.96" y="76.2" smashed="yes">
 <attribute name="NAME" x="57.15" y="77.6986" size="1.778" layer="95"/>
@@
 </instance>
 <instance part="GND9" gate="1" x="119.38" y="40.64"/>
+<instance part="X1" gate="G$1" x="86.36" y="71.12"/>
+<instance part="BAT1" gate="G$1" x="10.16" y="76.2"/>
 </instances>
 <busses>
@@
 <pinref part="GND2" gate="1" pin="GND"/>
 <wire x1="15.24" y1="76.2" x2="15.24" y2="71.12" width="0.1524" layer="91"/>
-<pinref part="BAT2" gate="G$1" pin="-"/>
+<pinref part="BAT1" gate="G$1" pin="-"/>
 </segment>
 <segment>
@@
 </segment>
 <segment>
-<pinref part="JP1" gate="G$1" pin="GND"/>
 <wire x1="73.66" y1="68.58" x2="71.12" y2="68.58" width="0.1524" layer="91"/>
 <wire x1="71.12" y1="68.58" x2="66.04" y2="68.58" width="0.1524" layer="91"/>
 <pinref part="GND5" gate="1" pin="GND"/>
+<pinref part="X1" gate="G$1" pin="GND"/>
+<wire x1="73.66" y1="68.58" x2="83.82" y2="68.58" width="0.1524" layer="91"/>
+<wire x1="83.82" y1="68.58" x2="83.82" y2="71.12" width="0.1524" layer="91"/>
 </segment>
 <segment>
@@
 <net name="N$6" class="0">
 <segment>
-<pinref part="IC1" gate="G$1" pin="(AIN1)PB1"/>
-<wire x1="55.88" y1="50.8" x2="63.5" y2="50.8" width="0.1524" layer="91"/>
 <pinref part="U4" gate="G$1" pin="SA0/SDO"/>
 <wire x1="17.78" y1="-10.16" x2="60.96" y2="-10.16" width="0.1524" layer="91"/>
 <wire x1="60.96" y1="-10.16" x2="63.5" y2="-10.16" width="0.1524" layer="91"/>
 <wire x1="63.5" y1="-10.16" x2="63.5" y2="17.78" width="0.1524" layer="91"/>
-<wire x1="63.5" y1="17.78" x2="63.5" y2="50.8" width="0.1524" layer="91"/>
 <pinref part="U$1" gate="G$1" pin="DO"/>
 <wire x1="76.2" y1="17.78" x2="63.5" y2="17.78" width="0.1524" layer="91"/>
+<pinref part="JP2" gate="G$1" pin="1"/>
+<wire x1="78.74" y1="48.26" x2="66.04" y2="48.26" width="0.1524" layer="91"/>
+<pinref part="IC1" gate="G$1" pin="(AIN0)PB0"/>
+<wire x1="55.88" y1="48.26" x2="63.5" y2="48.26" width="0.1524" layer="91"/>
+<wire x1="63.5" y1="48.26" x2="66.04" y2="48.26" width="0.1524" layer="91"/>
+<wire x1="63.5" y1="17.78" x2="63.5" y2="48.26" width="0.1524" layer="91"/>
 <junction x="63.5" y="17.78"/>
-<pinref part="JP2" gate="G$1" pin="2"/>
-<wire x1="78.74" y1="50.8" x2="63.5" y2="50.8" width="0.1524" layer="91"/>
-<junction x="63.5" y="50.8"/>
+<junction x="63.5" y="48.26"/>
 </segment>
 </net>
 <net name="N$7" class="0">
 <segment>
-<pinref part="IC1" gate="G$1" pin="(AIN0)PB0"/>
-<wire x1="55.88" y1="48.26" x2="66.04" y2="48.26" width="0.1524" layer="91"/>
 <pinref part="U4" gate="G$1" pin="SDA/SDI"/>
 <wire x1="17.78" y1="-7.62" x2="66.04" y2="-7.62" width="0.1524" layer="91"/>
@@
 <wire x1="66.04" y1="27.94" x2="66.04" y2="33.02" width="0.1524" layer="91"/>
 <pinref part="U$1" gate="G$1" pin="DI"/>
-<wire x1="66.04" y1="33.02" x2="66.04" y2="48.26" width="0.1524" layer="91"/>
 <wire x1="106.68" y1="12.7" x2="121.92" y2="12.7" width="0.1524" layer="91"/>
 <wire x1="121.92" y1="12.7" x2="121.92" y2="33.02" width="0.1524" layer="91"/>
 <wire x1="121.92" y1="33.02" x2="66.04" y2="33.02" width="0.1524" layer="91"/>
+<pinref part="JP2" gate="G$1" pin="2"/>
+<wire x1="78.74" y1="50.8" x2="66.04" y2="50.8" width="0.1524" layer="91"/>
+<pinref part="IC1" gate="G$1" pin="(AIN1)PB1"/>
+<wire x1="66.04" y1="50.8" x2="63.5" y2="50.8" width="0.1524" layer="91"/>
+<wire x1="55.88" y1="50.8" x2="63.5" y2="50.8" width="0.1524" layer="91"/>
+<wire x1="66.04" y1="33.02" x2="66.04" y2="50.8" width="0.1524" layer="91"/>
+<junction x="66.04" y="50.8"/>
 <junction x="66.04" y="33.02"/>
-<pinref part="JP2" gate="G$1" pin="1"/>
-<wire x1="78.74" y1="48.26" x2="66.04" y2="48.26" width="0.1524" layer="91"/>
-<junction x="66.04" y="48.26"/>
 </segment>
 </net>
 <net name="N$8" class="0">
 <segment>
-<pinref part="JP1" gate="G$1" pin="D-"/>
 <pinref part="R1" gate="G$1" pin="2"/>
 <wire x1="73.66" y1="76.2" x2="68.58" y2="76.2" width="0.1524" layer="91"/>
@@
 <wire x1="68.58" y1="78.74" x2="68.58" y2="76.2" width="0.1524" layer="91"/>
 <junction x="68.58" y="76.2"/>
+<pinref part="X1" gate="G$1" pin="D-"/>
+<wire x1="73.66" y1="76.2" x2="83.82" y2="76.2" width="0.1524" layer="91"/>
 </segment>
 </net>
@@
 <pinref part="P+2" gate="1" pin="VCC"/>
 <wire x1="-7.62" y1="76.2" x2="-2.54" y2="76.2" width="0.1524" layer="91"/>
-<pinref part="BAT2" gate="G$1" pin="+"/>
 <wire x1="-2.54" y1="76.2" x2="0" y2="76.2" width="0.1524" layer="91"/>
 <wire x1="5.08" y1="76.2" x2="0" y2="76.2" width="0.1524" layer="91"/>
@@
 <junction x="-35.56" y="-2.54"/>
 <junction x="5.08" y="33.02"/>
+<pinref part="BAT1" gate="G$1" pin="+"/>
 </segment>
 <segment>
@@
 <net name="N$2" class="0">
 <segment>
-<pinref part="JP1" gate="G$1" pin="D+"/>
 <pinref part="R2" gate="G$1" pin="2"/>
 <wire x1="73.66" y1="73.66" x2="68.58" y2="73.66" width="0.1524" layer="91"/>
 <wire x1="68.58" y1="73.66" x2="68.58" y2="71.12" width="0.1524" layer="91"/>
-</segment>
-</net>
+<wire x1="73.66" y1="73.66" x2="76.2" y2="73.66" width="0.1524" layer="91"/>
+<wire x1="76.2" y1="73.66" x2="76.2" y2="78.74" width="0.1524" layer="91"/>
+<pinref part="X1" gate="G$1" pin="D+"/>
+<wire x1="76.2" y1="78.74" x2="83.82" y2="78.74" width="0.1524" layer="91"/>
+</segment>
+</net>
