File: NanoLogger/NanoLogger.brd (EAGLE design)
At the start: 16.3 x 16.3 mm, 17 parts, among them U1 ATTINY2313-20MU, U4 LIS331

Commit message: Route looks better now
Parts:
- moved /RESET 17.2 mm to (7.80, 17.0)
- moved LED1 17.2 mm to (3.17, 12.3)
- moved SCK 17.2 mm to (9.96, 17.1)
- moved U4 17.2 mm to (13.3, 6.99)
- moved GND 17.2 mm to (6.71, 16.6)
- moved LED2 17.2 mm to (2.01, 9.45)
- moved MISO 17.2 mm to (11.0, 16.9)
- moved MOSI 17.2 mm to (12.0, 16.4)
- moved R1 17.2 mm to (13.5, 11.6)
- moved R3 17.2 mm to (3.40, 8.08)
- moved R5 17.2 mm to (8.89, 2.79)
- moved R6 17.2 mm to (4.90, 14.5)
- moved U$1 17.2 mm to (8.38, 4.93)
- moved U$2 17.2 mm to (8.43, 9.02)
- moved U1 17.2 mm to (9.07, 13.5)
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Routing:
- net ADI: track 28.2 -> 25.3 mm
- net ADO: track 24.2 -> 22.0 mm
- net ASCK: track 27.6 -> 26.0 mm
